Commit message: link updates

File: body.urdf (robot description, URDF)
Before this commit: robot robot, 3 links, 2 joints
Joints:
- joint Torso_BackLeg: origin xyz=1 0 0 rpy=0 0 0 -> xyz=1 0 1 rpy=0 0 0
- joint Torso_FrontLeg: child Torso -> FrontLeg; origin xyz=1 0 1 rpy=0 0 0 -> xyz=2 0 1 rpy=0 0 0; parent FrontLeg -> Torso

Commit message: last update

File: body.urdf (robot description, URDF)
Before this commit: robot robot, 3 links, 2 joints
Links:
- added link BackLowerLeg, mass 1; collision box size=0.2 0.2 1; visual box size=0.2 0.2 1
- added link FrontLowerLeg, mass 1; collision box size=0.2 0.2 1; visual box size=0.2 0.2 1
- added link LeftLeg, mass 1; collision box size=1 0.2 0.2; visual box size=1 0.2 0.2
- added link LeftLowerLeg, mass 1; collision box size=0.2 0.2 1; visual box size=0.2 0.2 1
- added link RightLeg, mass 1; collision box size=1 0.2 0.2; visual box size=1 0.2 0.2
- added link RightLowerLeg, mass 1; collision box size=0.2 0.2 1; visual box size=0.2 0.2 1
- link BackLeg: geometry collision box size=0.2 1 0.2; visual box size=0.2 1 0.2
- link FrontLeg: geometry collision box size=0.2 1 0.2; visual box size=0.2 1 0.2
Joints:
- added joint BackLeg_BackLowerLeg: type revolute, parent BackLeg, child BackLowerLeg, origin xyz=0 -1 0 rpy=0 0 0, axis 1 0 0, limit lower=-3.14159 upper=3.14159 effort=0.0 velocity=0.0
- added joint FrontLeg_FrontLowerLeg: type revolute, parent FrontLeg, child FrontLowerLeg, origin xyz=0 1 0 rpy=0 0 0, axis 1 0 0, limit lower=-3.14159 upper=3.14159 effort=0.0 velocity=0.0
- added joint LeftLeg_LeftLowerLeg: type revolute, parent LeftLeg, child LeftLowerLeg, origin xyz=-1 0 0 rpy=0 0 0, axis 0 1 0, limit lower=-3.14159 upper=3.14159 effort=0.0 velocity=0.0
- added joint RightLeg_RightLowerLeg: type revolute, parent RightLeg, child RightLowerLeg, origin xyz=1 0 0 rpy=0 0 0, axis 0 1 0, limit lower=-3.14159 upper=3.14159 effort=0.0 velocity=0.0
- added joint Torso_LeftLeg: type revolute, parent Torso, child LeftLeg, origin xyz=-0.5 0 1 rpy=0 0 0, axis 0 1 0, limit lower=-3.14159 upper=3.14159 effort=0.0 velocity=0.0
- added joint Torso_RightLeg: type revolute, parent Torso, child RightLeg, origin xyz=0.5 0 1 rpy=0 0 0, axis 0 1 0, limit lower=-3.14159 upper=3.14159 effort=0.0 velocity=0.0
- joint Torso_BackLeg: axis 0 1 0 -> 1 0 0; origin xyz=1 0 1 rpy=0 0 0 -> xyz=0 -0.5 1 rpy=0 0 0
- joint Torso_FrontLeg: axis 0 1 0 -> 1 0 0; origin xyz=2 0 1 rpy=0 0 0 -> xyz=0 0.5 1 rpy=0 0 0

Commit message: legs

File: body.urdf (robot description, URDF)
Before this commit: robot robot, 9 links, 8 joints
Links:
- link LeftLeg: geometry collision box size=0.2 1 0.2; visual box size=0.2 1 0.2
- link RightLeg: geometry collision box size=0.2 1 0.2; visual box size=0.2 1 0.2
- link Torso: geometry collision box size=3 1 1; visual box size=3 1 1
Joints:
- joint BackLeg_BackLowerLeg: origin xyz=0 -1 0 rpy=0 0 0 -> xyz=0.5 -1 0 rpy=0 0 0
- joint LeftLeg_LeftLowerLeg: axis 0 1 0 -> 1 0 0; origin xyz=-1 0 0 rpy=0 0 0 -> xyz=0 1 0 rpy=0 0 0
- joint RightLeg_RightLowerLeg: origin xyz=1 0 0 rpy=0 0 0 -> xyz=-0.5 -1 0 rpy=0 0 0
- joint Torso_BackLeg: origin xyz=0 -0.5 1 rpy=0 0 0 -> xyz=0.5 -0.5 1 rpy=0 0 0
- joint Torso_FrontLeg: origin xyz=0 0.5 1 rpy=0 0 0 -> xyz=0.5 0.5 1 rpy=0 0 0
- joint Torso_LeftLeg: axis 0 1 0 -> 1 0 0; origin xyz=-0.5 0 1 rpy=0 0 0 -> xyz=-0.5 0.5 1 rpy=0 0 0
- joint Torso_RightLeg: origin xyz=0.5 0 1 rpy=0 0 0 -> xyz=-0.5 -0.5 1 rpy=0 0 0

Commit message: finished

File: body.urdf (robot description, URDF)
Before this commit: robot robot, 9 links, 8 joints
Links:
- link Torso: geometry collision box size=3 1 0.75; visual box size=3 1 0.75
Joints:
- joint BackLeg_BackLowerLeg: axis 1 0 0 -> 0 1 0
- joint FrontLeg_FrontLowerLeg: axis 1 0 0 -> 0 1 0
- joint LeftLeg_LeftLowerLeg: axis 1 0 0 -> 0 1 0
- joint Torso_BackLeg: axis 1 0 0 -> 0 1 0
- joint Torso_FrontLeg: axis 1 0 0 -> 0 1 0
- joint Torso_LeftLeg: axis 1 0 0 -> 0 1 0

Commit message: first try

File: body.urdf (robot description, URDF)
Before this commit: robot robot, 9 links, 8 joints
Links:
- removed link BackLeg
- removed link BackLowerLeg
- removed link FrontLeg
- removed link FrontLowerLeg
- removed link LeftLeg
- removed link LeftLowerLeg
- removed link RightLeg
- removed link RightLowerLeg
- removed link Torso
- added link link0, mass 1; collision box size=1 1 1; visual box size=1 1 1
- added link link1, mass 1; collision box size=1 2 3; visual box size=1 2 3
- added link link2, mass 1; collision box size=5 4 4; visual box size=5 4 4
- added link link3, mass 1; collision box size=3 5 5; visual box size=3 5 5
- added link link4, mass 1; collision box size=4 3 4; visual box size=4 3 4
- added link link5, mass 1; collision box size=3 3 2; visual box size=3 3 2
Joints:
- removed joint BackLeg_BackLowerLeg
- removed joint FrontLeg_FrontLowerLeg
- removed joint LeftLeg_LeftLowerLeg
- removed joint RightLeg_RightLowerLeg
- removed joint Torso_BackLeg
- removed joint Torso_FrontLeg
- removed joint Torso_LeftLeg
- removed joint Torso_RightLeg
- added joint link0: type revolute, parent link0, child link1, origin xyz=0 0.5 2.5 rpy=0 0 0, axis 1 0 0, limit lower=-3.14159 upper=3.14159 effort=0.0 velocity=0.0
- added joint link1_link2: type revolute, parent link1, child link2, origin xyz=0 2 2.5 rpy=0 0 0, axis 1 0 0, limit lower=-3.14159 upper=3.14159 effort=0.0 velocity=0.0
- added joint link2_link3: type revolute, parent link2, child link3, origin xyz=0 4 2.5 rpy=0 0 0, axis 1 0 0, limit lower=-3.14159 upper=3.14159 effort=0.0 velocity=0.0
- added joint link3_link4: type revolute, parent link3, child link4, origin xyz=0 5 2.5 rpy=0 0 0, axis 1 0 0, limit lower=-3.14159 upper=3.14159 effort=0.0 velocity=0.0
- added joint link4_link5: type revolute, parent link4, child link5, origin xyz=0 3 2.5 rpy=0 0 0, axis 1 0 0, limit lower=-3.14159 upper=3.14159 effort=0.0 velocity=0.0
- added joint link5_link6: type revolute, parent link5, child link6, origin xyz=0 3 2.5 rpy=0 0 0, axis 1 0 0, limit lower=-3.14159 upper=3.14159 effort=0.0 velocity=0.0

Commit message: fixed the snake!

File: body.urdf (robot description, URDF)
Before this commit: robot robot, 6 links, 6 joints
Links:
- link link1: geometry collision box size=2 4 1; visual box size=2 4 1
- link link2: geometry collision box size=1 3 4; visual box size=1 3 4
- link link3: geometry collision box size=4 3 2; visual box size=4 3 2
- link link4: geometry collision box size=2 1 2; visual box size=2 1 2
- link link5: geometry collision box size=3 2 3; visual box size=3 2 3
Joints:
- removed joint link0
- removed joint link5_link6
- added joint link0_link1: type revolute, parent link0, child link1, origin xyz=0 0.5 2 rpy=0 0 0, axis 1 0 0, limit lower=-3.14159 upper=3.14159 effort=0.0 velocity=0.0
- joint link1_link2: origin xyz=0 2 2.5 rpy=0 0 0 -> xyz=0 4 2 rpy=0 0 0
- joint link2_link3: origin xyz=0 4 2.5 rpy=0 0 0 -> xyz=0 3 2 rpy=0 0 0
- joint link3_link4: origin xyz=0 5 2.5 rpy=0 0 0 -> xyz=0 3 2 rpy=0 0 0
- joint link4_link5: origin xyz=0 3 2.5 rpy=0 0 0 -> xyz=0 1 2 rpy=0 0 0

Commit message: playing with sizing

File: body.urdf (robot description, URDF)
Before this commit: robot robot, 6 links, 5 joints
Links:
- removed link link5
- link link1: geometry collision box size=2 3 1.2; visual box size=2 3 1.2
- link link2: geometry collision box size=2 3 1.2; visual box size=2 3 1.2
- link link3: geometry collision box size=1 3 2.2; visual box size=1 3 2.2
- link link4: geometry collision box size=2 1 3.2; visual box size=2 1 3.2
Joints:
- removed joint link4_link5
- joint link0_link1: axis 1 0 0 -> 0 0 1; origin xyz=0 0.5 2 rpy=0 0 0 -> xyz=0 0.5 2.5 rpy=0 0 0
- joint link1_link2: axis 1 0 0 -> 0 0 1; origin xyz=0 4 2 rpy=0 0 0 -> xyz=0 3 2.5 rpy=0 0 0
- joint link2_link3: axis 1 0 0 -> 0 0 1; origin xyz=0 3 2 rpy=0 0 0 -> xyz=0 3 2.5 rpy=0 0 0
- joint link3_link4: axis 1 0 0 -> 0 0 1; origin xyz=0 3 2 rpy=0 0 0 -> xyz=0 3 2.5 rpy=0 0 0

Commit message: trying colors

File: body.urdf (robot description, URDF)
Before this commit: robot robot, 5 links, 4 joints
Links:
- added link link5, mass 1; collision box size=2 1 1; visual box size=2 1 1
- added link link6, mass 1; collision box size=1 2 1; visual box size=1 2 1
- link link1: geometry collision box size=2 2 1; visual box size=2 2 1
- link link2: geometry collision box size=1 1 1; visual box size=1 1 1
- link link3: geometry collision box size=1 2 1; visual box size=1 2 1
- link link4: geometry collision box size=2 1 2; visual box size=2 1 2
Joints:
- added joint link4_link5: type revolute, parent link4, child link5, origin xyz=0 1 0.5 rpy=0 0 0, axis 0 0 1, limit lower=-3.14159 upper=3.14159 effort=0.0 velocity=0.0
- added joint link5_link6: type revolute, parent link5, child link6, origin xyz=0 1 0.5 rpy=0 0 0, axis 0 0 1, limit lower=-3.14159 upper=3.14159 effort=0.0 velocity=0.0
- joint link0_link1: origin xyz=0 0.5 2.5 rpy=0 0 0 -> xyz=0 0.5 0.5 rpy=0 0 0
- joint link1_link2: origin xyz=0 3 2.5 rpy=0 0 0 -> xyz=0 2 0.5 rpy=0 0 0
- joint link2_link3: origin xyz=0 3 2.5 rpy=0 0 0 -> xyz=0 1 0.5 rpy=0 0 0
- joint link3_link4: origin xyz=0 3 2.5 rpy=0 0 0 -> xyz=0 2 0.5 rpy=0 0 0

Commit message: finished snakes

File: body.urdf (robot description, URDF)
Before this commit: robot robot, 7 links, 6 joints
Links:
- added link link7, mass 1; collision box size=2 1 1; visual box size=2 1 1
- added link link8, mass 1; collision box size=1 2 1; visual box size=1 2 1
- link link1: geometry collision box size=1 1 2; visual box size=1 1 2
- link link2: geometry collision box size=2 2 1; visual box size=2 2 1
- link link3: geometry collision box size=2 2 2; visual box size=2 2 2
- link link4: geometry collision box size=1 1 1; visual box size=1 1 1
- link link5: geometry collision box size=2 2 2; visual box size=2 2 2
- link link6: geometry collision box size=1 1 1; visual box size=1 1 1
Joints:
- added joint link6_link7: type revolute, parent link6, child link7, origin xyz=0 1 0.5 rpy=0 0 0, axis 0 0 1, limit lower=-3.14159 upper=3.14159 effort=0.0 velocity=0.0
- added joint link7_link8: type revolute, parent link7, child link8, origin xyz=0 1 0.5 rpy=0 0 0, axis 0 0 1, limit lower=-3.14159 upper=3.14159 effort=0.0 velocity=0.0
- joint link1_link2: origin xyz=0 2 0.5 rpy=0 0 0 -> xyz=0 1 0.5 rpy=0 0 0
- joint link2_link3: origin xyz=0 1 0.5 rpy=0 0 0 -> xyz=0 2 0.5 rpy=0 0 0
- joint link5_link6: origin xyz=0 1 0.5 rpy=0 0 0 -> xyz=0 2 0.5 rpy=0 0 0
